File: PCB/Camera Stand/Siren.kicad_sch (KiCad schematic)
At the start: 5 parts, among them Q1 PN2222A

Commit message: 3.3v error in PCB
Parts:
- gave numbers to parts that had none: 1
Changed lines of the file:
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@@
   (symbol (lib_id "Relay:FINDER-36.11") (at 187.96 100.33 0) (unit 1)
     (in_bom yes) (on_board yes) (fields_autoplaced)
-    (property "Reference" "K?" (id 0) (at 199.39 99.0599 0)
+    (property "Reference" "K1" (id 0) (at 199.39 99.0599 0)
       (effects (font (size 1.27 1.27)) (justify left))
     )

Commit message: 12v to siren
Connections:
- net VCC renamed VCC1
- net VCC1: no longer Q1.3 (C)
- new net VCC2: Q1.3 (C)
Changed lines of the file:
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@@
 (kicad_sch (version 20211123) (generator eeschema)
   (paper "A4")
-  (junction (at 171.45 63.5) (diameter 0) (color 0 0 0 0)
-  )
   (junction (at 171.45 92.71) (diameter 0) (color 0 0 0 0)
   )
@@
   )
   (junction (at 171.45 107.95) (diameter 0) (color 0 0 0 0)
-  )
-  (wire (pts (xy 171.45 63.5) (xy 195.58 63.5))
-    (stroke (width 0) (type default) (color 0 0 0 0))
   )
   (wire (pts (xy 152.4 76.2) (xy 163.83 76.2))
@@
     (stroke (width 0) (type default) (color 0 0 0 0))
   )
+  (wire (pts (xy 138.43 58.42) (xy 195.58 58.42))
+    (stroke (width 0) (type default) (color 0 0 0 0))
+  )
   (wire (pts (xy 91.44 76.2) (xy 144.78 76.2))
+    (stroke (width 0) (type default) (color 0 0 0 0))
+  )
+  (wire (pts (xy 138.43 68.58) (xy 138.43 58.42))
     (stroke (width 0) (type default) (color 0 0 0 0))
   )
@@
     (stroke (width 0) (type default) (color 0 0 0 0))
   )
-  (wire (pts (xy 171.45 81.28) (xy 171.45 92.71))
+  (wire (pts (xy 195.58 58.42) (xy 195.58 92.71))
     (stroke (width 0) (type default) (color 0 0 0 0))
   )
-  (wire (pts (xy 195.58 63.5) (xy 195.58 92.71))
+  (wire (pts (xy 171.45 81.28) (xy 171.45 92.71))
     (stroke (width 0) (type default) (color 0 0 0 0))
   )
@@
     (stroke (width 0) (type default) (color 0 0 0 0))
   )
+  (wire (pts (xy 91.44 68.58) (xy 138.43 68.58))
+    (stroke (width 0) (type default) (color 0 0 0 0))
+  )
   (wire (pts (xy 171.45 63.5) (xy 171.45 71.12))
     (stroke (width 0) (type default) (color 0 0 0 0))
@@
   (wire (pts (xy 91.44 72.39) (xy 142.24 72.39))
     (stroke (width 0) (type default) (color 0 0 0 0))
+  )
+  (hierarchical_label "VCC1" (shape input) (at 91.44 68.58 180)
+    (effects (font (size 1.27 1.27)) (justify right))
   )
   (hierarchical_label "S0" (shape input) (at 91.44 76.2 180)
@@
     (effects (font (size 1.27 1.27)) (justify right))
   )
-  (hierarchical_label "VCC" (shape input) (at 91.44 72.39 180)
+  (hierarchical_label "VCC2" (shape input) (at 91.44 72.39 180)
     (effects (font (size 1.27 1.27)) (justify right))
   )
